File: Documents/Eagle/ardOnTimer.sch (EAGLE design)
At the start: 15 parts

Commit message: Switched DI12<->DI13
Connections:
- removed net N$19: B1.D13, SV3.SIG
- new net N$17: B1.D12, SV3.SIG
- net N$2: now also B1.D13; no longer B1.D12
Changed lines of the file:
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@@
-</segment>
-</net>
-<net name="N$19" class="0">
-<segment>
-<pinref part="SV3" gate="G$1" pin="SIG"/>
-<wire x1="170.18" y1="63.5" x2="241.3" y2="63.5" width="0.1524" layer="91"/>
-<pinref part="B1" gate="G$1" pin="D13"/>
-<wire x1="147.32" y1="101.6" x2="170.18" y2="101.6" width="0.1524" layer="91"/>
-<wire x1="170.18" y1="101.6" x2="170.18" y2="63.5" width="0.1524" layer="91"/>
 </segment>
 </net>
 <net name="N$2" class="0">
 <segment>
-<pinref part="B1" gate="G$1" pin="D12"/>
-<wire x1="147.32" y1="104.14" x2="236.22" y2="104.14" width="0.1524" layer="91"/>
-<wire x1="236.22" y1="104.14" x2="236.22" y2="93.98" width="0.1524" layer="91"/>
+<pinref part="B1" gate="G$1" pin="D13"/>
+<wire x1="147.32" y1="101.6" x2="236.22" y2="101.6" width="0.1524" layer="91"/>
 <pinref part="SG1" gate="G$1" pin="1"/>
+<wire x1="236.22" y1="101.6" x2="236.22" y2="93.98" width="0.1524" layer="91"/>
 </segment>
 </net>
+<net name="N$17" class="0">
+<segment>
+<pinref part="B1" gate="G$1" pin="D12"/>
+<wire x1="147.32" y1="104.14" x2="233.68" y2="104.14" width="0.1524" layer="91"/>
+<wire x1="233.68" y1="104.14" x2="233.68" y2="63.5" width="0.1524" layer="91"/>
+<pinref part="SV3" gate="G$1" pin="SIG"/>
+<wire x1="233.68" y1="63.5" x2="241.3" y2="63.5" width="0.1524" layer="91"/>
+</segment>
+</net>

Commit message: Forgot resistor in schematics. Updated readme.
Parts:
- added R7: 100R, rcl:R-EU_0204/7
Connections:
- new net N$18: R7.2, SG1.2
- net N$1: now also R7.1; no longer SG1.2
Changed lines of the file:
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@@
 <part name="SV3" library="myLib-01-Headers" deviceset="KY-019_3-PIN_FEMALE_HEADER" device="ANGLED_W_MOUNT_HOLES"/>
 <part name="SG1" library="buzzer" library_urn="urn:adsk.eagle:library:113" deviceset="F/CM12P" device="" package3d_urn="urn:adsk.eagle:package:5265/1"/>
+<part name="R7" library="rcl" library_urn="urn:adsk.eagle:library:334" deviceset="R-EU_" device="0204/7" package3d_urn="urn:adsk.eagle:package:23498/2" value="100R"/>
 </parts>
 <sheets>
@@
 <attribute name="NAME" x="245.11" y="93.98" size="1.778" layer="95" rot="R270"/>
 <attribute name="VALUE" x="238.76" y="85.09" size="1.778" layer="96" rot="R270"/>
+</instance>
+<instance part="R7" gate="G$1" x="213.36" y="71.12" smashed="yes" rot="R90">
+<attribute name="NAME" x="211.8614" y="67.31" size="1.778" layer="95" rot="R90"/>
+<attribute name="VALUE" x="216.662" y="67.31" size="1.778" layer="96" rot="R90"/>
 </instance>
 </instances>
@@
 <junction x="175.26" y="157.48"/>
 <pinref part="SV3" gate="G$1" pin="GND"/>
-<wire x1="175.26" y1="58.42" x2="236.22" y2="58.42" width="0.1524" layer="91"/>
-<wire x1="236.22" y1="58.42" x2="241.3" y2="58.42" width="0.1524" layer="91"/>
+<wire x1="175.26" y1="58.42" x2="213.36" y2="58.42" width="0.1524" layer="91"/>
+<wire x1="213.36" y1="58.42" x2="241.3" y2="58.42" width="0.1524" layer="91"/>
 <wire x1="175.26" y1="185.42" x2="175.26" y2="200.66" width="0.1524" layer="91"/>
 <wire x1="175.26" y1="200.66" x2="309.88" y2="200.66" width="0.1524" layer="91"/>
@@
 <wire x1="309.88" y1="200.66" x2="309.88" y2="185.42" width="0.1524" layer="91"/>
 <junction x="309.88" y="185.42"/>
-<wire x1="236.22" y1="86.36" x2="236.22" y2="58.42" width="0.1524" layer="91"/>
-<junction x="236.22" y="58.42"/>
-<pinref part="SG1" gate="G$1" pin="2"/>
+<pinref part="R7" gate="G$1" pin="1"/>
+<wire x1="213.36" y1="66.04" x2="213.36" y2="58.42" width="0.1524" layer="91"/>
+<junction x="213.36" y="58.42"/>
 </segment>
 </net>
@@
 </segment>
 </net>
+<net name="N$18" class="0">
+<segment>
+<pinref part="SG1" gate="G$1" pin="2"/>
+<wire x1="236.22" y1="86.36" x2="236.22" y2="81.28" width="0.1524" layer="91"/>
+<wire x1="236.22" y1="81.28" x2="213.36" y2="81.28" width="0.1524" layer="91"/>
+<pinref part="R7" gate="G$1" pin="2"/>
+<wire x1="213.36" y1="81.28" x2="213.36" y2="76.2" width="0.1524" layer="91"/>
+</segment>
+</net>
