File: KiCad/ardOnTimer-atmega/ATmega328.kicad_sch (KiCad schematic)
At the start: 15 parts, among them J1 FTDI, J2 Power in, U1 AMS1117-5.0, U2 ATmega328P-PU, Y1 16MHz

Commit message: kicad
Other:
- title: (none) -> ardOnTImer-ATmega
Changed lines of the file:
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@@
 (kicad_sch (version 20211123) (generator eeschema)
   (paper "A4")
+  (title_block
+    (title "ardOnTImer-ATmega")
+    (date "2022-09-09")
+    (rev "0.2")
+  )
   (junction (at 220.98 134.62) (diameter 0) (color 0 0 0 0)
   )

Commit message: kicad v0.3
Parts:
- removed C5: 100n, My_Misc:C_Disc_D3.0mm_W1.6mm_P2.50mm_larg, symbol Device:C
- removed J1: FTDI, My_Headers:6-pin FTDI Programmer PinSocket large, symbol My_Headers:6-pin_FTDI_header
- added C3, C4, C7: 100n, My_Misc:C_Disc_D4.3mm_W1.9mm_P5.00mm_large, symbol Device:C
- added J3: FTDI, My_Headers:6-pin FTDI Programmer PinSocket large, symbol My_Headers:6-pin_FTDI_header
- added JP1: FTDI Power, My_Parts:Jumper_1x02_P2.54mm_large, symbol Jumper:Jumper_2_Open
- renumbered C4 to C2, C2 to C5, C3 to C6, R1 to R7, U1 to U3, U2 to U4
Connections:
- net +5V: now also C3.1, C4.2, C7.2, JP1.2 (B)
- net D0/Rx: now also J3.4 (Tx)
- net D1/Tx: now also J3.5 (Rx)
- net GND: now also C3.2, C4.1, J3.1 (GND)
- new net: C7.1, J3.6 (DTR)
- new net: J3.3 (VCC), JP1.1 (A)
